Commit message: robot sim gazebo

File: description/robot.urdf.xacro (robot description, xacro)
@@ -2,3 +2,4 @@
 <robot xmlns:xacro="http://www.ros.org/wiki/xacro"  name="robot">
     <xacro:include filename="robot_core.xacro"/>
+    <xacro:include filename="gazebo_control.xacro"/>
 </robot>

File: description/robot_core.xacro (robot description, xacro)
@@ -1,17 +1,18 @@
 <?xml version="1.0"?>
 <robot xmlns:xacro="http://www.ros.org/wiki/xacro">
+    <xacro:include filename="inertial_macros.xacro"/>
     <material name="white">
         <color rgba="1 1 1 1"/>
     </material>
-     <material name="orange">
+    <material name="orange">
         <color rgba="1 0.3 0.1 1"/>
     </material>
-     <material name="blue">
+    <material name="blue">
         <color rgba="0.2 0.2 1 1"/>
     </material>
-     <material name="black">
+    <material name="black">
         <color rgba="0 0 0 1"/>
     </material>
-    <!--BASE LINK-->
+        <!--BASE LINK-->
     <link name="base_link">
     </link>
@@ -30,62 +31,118 @@
             <material name="white"/>
         </visual>
+         <collision>
+            <origin xyz="0.2 0 0.053"/>
+            <geometry>
+                <box size="0.4 0.3 0.106"/>
+            </geometry>
+        </collision>
+        <xacro:inertial_box mass="0.5" x="0.4" y="0.3" z="0.106">
+            <origin xyz="0.2 0 0.053" rpy="0 0 0"/>
+        </xacro:inertial_box>
     </link>
-     <!--LEFT WHELS-->
-     <joint name="left_wheel_joint" type="continuous">
+    <gazebo reference="chassis">
+        <material>Gazebo/White</material>
+    </gazebo>
+        <!--LEFT WHELS-->
+    <joint name="left_wheel_joint" type="continuous">
         <parent link="base_link"/>
         <child link="left_wheel"/>
-        <origin xyz="0.1323 0.15 0" rpy="-${pi/2} 0 0"/>
+        <origin xyz="0.1323 0.18 0.0235" rpy="-${pi/2} 0 0"/>
         <axis xyz="0 0 1"/>
-     </joint>
+    </joint>
     <link name="left_wheel">
         <visual>
             <geometry>
-                <cylinder radius="0.068" length="0.067"/>
+                <cylinder radius="0.068" length="0.06"/>
             </geometry>
             <material name="blue"/>
         </visual>
+        <collision>
+            <geometry>
+                <cylinder radius="0.068" length="0.06"/>
+            </geometry>
+        </collision>
+        <xacro:inertial_cylinder mass="0.1" length="0.06" radius="0.068">
+            <origin xyz="0 0 0" rpy="0 0 0"/>
+        </xacro:inertial_cylinder>
     </link>
-      <joint name="left_wheel_joint1" type="continuous">
+    <gazebo reference="left_wheel">
+        <material>Gazebo/Blue</material>
+    </gazebo>
+    <joint name="left_wheel_joint1" type="continuous">
         <parent link="base_link"/>
         <child link="left_wheel1"/>
-        <origin xyz="-0.1323 0.18 0" rpy="-${pi/2} 0 0"/>
+        <origin xyz="-0.1323 0.18 0.0235" rpy="-${pi/2} 0 0"/>
         <axis xyz="0 0 1"/>
-     </joint>
+    </joint>
     <link name="left_wheel1">
         <visual>
             <geometry>
-                <cylinder radius="0.068" length="0.067"/>
+                <cylinder radius="0.068" length="0.06"/>
             </geometry>
             <material name="blue"/>
         </visual>
+        <collision>
+            <geometry>
+                <cylinder radius="0.068" length="0.06"/>
+            </geometry>
+        </collision>
+        <xacro:inertial_cylinder mass="0.1" length="0.06" radius="0.068">
+            <origin xyz="0 0 0" rpy="0 0 0"/>
+        </xacro:inertial_cylinder>
     </link>
-     <!--RIGHT WHELS-->
-     <joint name= "right_wheel_joint" type="continuous">
+    <gazebo reference="left_wheel1">
+        <material>Gazebo/Blue</material>
+    </gazebo>
+        <!--RIGHT WHELS-->
+    <joint name= "right_wheel_joint" type="continuous">
         <parent link="base_link"/>
         <child link="right_wheel"/>
-        <origin xyz="0.1323 -0.15 0" rpy="${pi/2} 0 0"/>
+        <origin xyz="0.1323 -0.18 0.0235" rpy="${pi/2} 0 0"/>
         <axis xyz="0 0 -1"/>
-     </joint>
+    </joint>
     <link name="right_wheel">
         <visual>
             <geometry>
-                <cylinder radius="0.068" length="0.067"/>
+                <cylinder radius="0.068" length="0.06"/>
             </geometry>
             <material name="blue"/>
         </visual>
+         <collision>
+            <geometry>
+                <cylinder radius="0.068" length="0.06"/>
+            </geometry>
+        </collision>
+        <xacro:inertial_cylinder mass="0.1" length="0.06" radius="0.068">
+            <origin xyz="0 0 0" rpy="0 0 0"/>
+        </xacro:inertial_cylinder>
     </link>
-     <joint name= "right_wheel_joint1" type="continuous">
+    <gazebo reference="right_wheel">
+        <material>Gazebo/Blue</material>
+    </gazebo>
+    <joint name= "right_wheel_joint1" type="continuous">
         <parent link="base_link"/>
         <child link="right_wheel1"/>
-        <origin xyz="-0.1323 -0.15 0" rpy="${pi/2} 0 0"/>
+        <origin xyz="-0.1323 -0.18 0.0235" rpy="${pi/2} 0 0"/>
         <axis xyz="0 0 -1"/>
-     </joint>
+    </joint>
     <link name="right_wheel1">
         <visual>
             <geometry>
-                <cylinder radius="0.068" length="0.067"/>
+                <cylinder radius="0.068" length="0.06"/>
             </geometry>
             <material name="blue"/>
         </visual>
+        <collision>
+            <geometry>
+                <cylinder radius="0.068" length="0.06"/>
+            </geometry>
+        </collision>
+        <xacro:inertial_cylinder mass="0.1" length="0.06" radius="0.068">
+            <origin xyz="0 0 0" rpy="0 0 0"/>
+        </xacro:inertial_cylinder>
     </link>
+    <gazebo reference="right_wheel1">
+        <material>Gazebo/Blue</material>
+    </gazebo>
 </robot>

Commit message: add laser xacro

File: description/robot.urdf.xacro (robot description, xacro)
@@ -3,3 +3,4 @@
     <xacro:include filename="robot_core.xacro"/>
     <xacro:include filename="gazebo_control.xacro"/>
+    <xacro:include filename="lidar.xacro"/>
 </robot>

File: description/robot_core.xacro (robot description, xacro)
@@ -12,4 +12,7 @@
     </material>
     <material name="black">
+        <color rgba="0 0 0 1"/>
+    </material>
+     <material name="red">
         <color rgba="0 0 0 1"/>
     </material>
