Commit message: restore git config

File: description/lidar.xacro (robot description, xacro)
@@ -4,10 +4,10 @@
     <parent link="chassis"/>
     <child link="laser_frame"/>
-    <origin xyz="0 0 0.106" rpy="0 0 0"/>
+    <origin xyz="0.2 0 0.126" rpy="0 0 0"/>
 </joint>
 <link name="laser_frame">
     <visual>
         <geometry>
-            <cylinder radius="0.068" length="0.06"/>
+            <cylinder radius="0.068" length="0.04"/>
         </geometry>
         <material name="red"/>
@@ -15,10 +15,38 @@
     <collision>
         <geometry>
-            <cylinder radius="0.068" length="0.06"/>
+            <cylinder radius="0.068" length="0.04"/>
         </geometry>
     </collision>
-    <xacro:inertial_cylinder mass="0.1" length="0.06" radius="0.068">
+    <xacro:inertial_cylinder mass="0.1" length="0.04" radius="0.068">
         <origin xyz="0 0 0" rpy="0 0 0"/>
     </xacro:inertial_cylinder>
 </link>
+<gazebo reference="laser_frame">
+        <material>Gazebo/Red</material>
+        <sensor name="laser" type="ray">
+            <pose> 0 0 0 0 0 0 </pose>
+            <visualize>true</visualize>
+            <update_rate>10</update_rate>
+            <ray>
+                <scan>
+                    <horizontal>
+                        <samples>360</samples>
+                        <min_angle>-3.14</min_angle>
+                        <max_angle>3.14</max_angle>
+                    </horizontal>
+                </scan>
+                <range>
+                    <min>0.3</min>
+                    <max>12</max>
+                </range>
+            </ray>
+            <plugin name="laser_controller" filename="libgazebo_ros_ray_sensor.so">
+                <ros>
+                    <argument>~/out:=scan</argument>
+                </ros>
+                <output_type>sensor_msgs/LaserScan</output_type>
+                <frame_name>laser_frame</frame_name>
+            </plugin>
+        </sensor>
+    </gazebo>
 </robot>
