Commit message: add 4 wheels dif driver config

File: description/gazebo_control.xacro (robot description, xacro)
@@ -2,10 +2,10 @@
 <robot xmlns:xacro="http://www.ros.org/wiki/xacro">
     <gazebo>
-        <plugin name='diff_drive' filename='libgazebo_ros_diff_drive.so'>
+        <plugin name="diff_drive" filename="libgazebo_ros_diff_drive.so">
             <!-- Wheel Information -->
-            <left_joint>left_wheel_joint</left_joint>
-            <right_joint>right_wheel_joint</right_joint>
-             <left_joint1>left_wheel_joint1</left_joint1>
-            <right_joint1>right_wheel_joint1</right_joint1>
+            <left_front_joint>left_front_wheel_joint</left_joint>
+            <right_front_joint>right_front_wheel_joint</right_joint>
+            <left_back_joint>left_back_wheel_joint</left_joint>
+            <right_back_joint>right_back_wheel_joint</right_joint>
             <wheel_separation>0.36</wheel_separation>
             <wheel_diameter>0.136</wheel_diameter>

File: description/robot.urdf.xacro (robot description, xacro)
@@ -1,7 +1,12 @@
 <?xml version="1.0"?>
 <robot xmlns:xacro="http://www.ros.org/wiki/xacro"  name="robot">
+    <xacro:args name="use_ros2_control" default="true"/>
     <xacro:include filename="robot_core.xacro"/>
+    <xacro:if value="${arg use_ros2_control}">
     <xacro:include filename="ros2_control.xacro"/>
+    </xacro:if>
+    <xacro:unless value="${arg use_ros2_control}">
     <xacro:include filename="gazebo_control.xacro"/>
+    </xacro:unless>
     <xacro:include filename="lidar.xacro"/>
     <xacro:include filename="camera.xacro"/>

File: description/robot_core.xacro (robot description, xacro)
@@ -48,11 +48,11 @@
     </gazebo>
         <!--LEFT WHELS-->
-    <joint name="left_wheel_joint" type="continuous">
+    <joint name="left_front_wheel_joint" type="continuous">
         <parent link="base_link"/>
-        <child link="left_wheel"/>
+        <child link="left_front_wheel"/>
         <origin xyz="0.1323 0.18 0.0235" rpy="-${pi/2} 0 0"/>
         <axis xyz="0 0 1"/>
     </joint>
-    <link name="left_wheel">
+    <link name="left_front_wheel">
         <visual>
             <geometry>
@@ -70,14 +70,14 @@
         </xacro:inertial_cylinder>
     </link>
-    <gazebo reference="left_wheel">
+    <gazebo reference="left_front_wheel">
         <material>Gazebo/Blue</material>
     </gazebo>
-    <joint name="left_wheel_joint1" type="continuous">
+    <joint name="left_back_wheel_joint" type="continuous">
         <parent link="base_link"/>
-        <child link="left_wheel1"/>
+        <child link="left_back_wheel"/>
         <origin xyz="-0.1323 0.18 0.0235" rpy="-${pi/2} 0 0"/>
         <axis xyz="0 0 1"/>
     </joint>
-    <link name="left_wheel1">
+    <link name="left_back_wheel">
         <visual>
             <geometry>
@@ -95,15 +95,15 @@
         </xacro:inertial_cylinder>
     </link>
-    <gazebo reference="left_wheel1">
+    <gazebo reference="left_back_wheel">
         <material>Gazebo/Blue</material>
     </gazebo>
         <!--RIGHT WHELS-->
-    <joint name= "right_wheel_joint" type="continuous">
+    <joint name= "right_front_wheel_joint" type="continuous">
         <parent link="base_link"/>
-        <child link="right_wheel"/>
+        <child link="right_front_wheel"/>
         <origin xyz="0.1323 -0.18 0.0235" rpy="${pi/2} 0 0"/>
         <axis xyz="0 0 -1"/>
     </joint>
-    <link name="right_wheel">
+    <link name="right_front_wheel">
         <visual>
             <geometry>
@@ -121,14 +121,14 @@
         </xacro:inertial_cylinder>
     </link>
-    <gazebo reference="right_wheel">
+    <gazebo reference="right_front_wheel">
         <material>Gazebo/Blue</material>
     </gazebo>
-    <joint name= "right_wheel_joint1" type="continuous">
+    <joint name= "right_back_wheel_joint" type="continuous">
         <parent link="base_link"/>
-        <child link="right_wheel1"/>
+        <child link="right_back_wheel"/>
         <origin xyz="-0.1323 -0.18 0.0235" rpy="${pi/2} 0 0"/>
         <axis xyz="0 0 -1"/>
     </joint>
-    <link name="right_wheel1">
+    <link name="right_back_wheel">
         <visual>
             <geometry>
@@ -146,5 +146,5 @@
         </xacro:inertial_cylinder>
     </link>
-    <gazebo reference="right_wheel1">
+    <gazebo reference="right_back_wheel">
         <material>Gazebo/Blue</material>
     </gazebo>

File: description/ros2_control.xacro (robot description, xacro)
@@ -5,17 +5,33 @@
             <plugin>gazebo_ros2_control/GazeboSystem</plugin>
         </hardware>
-        <joint name="left_wheel_joint">
-            <comand_interface name="velocity">
-                <param name="min">10</param>
+        <joint name="left_front_wheel_joint">
+            <command_interface name="velocity">
+                <param name="min">-10</param>
                 <param name="max">10</param>
-            </comand_interface>
+            </command_interface>
             <state_interface name="velocity"/>
             <state_interface name="position"/>
         </joint>
-             <joint name="right_wheel_joint">
-            <comand_interface name="velocity">
-                <param name="min">10</param>
+        <joint name="left_back_wheel_joint">
+            <command_interface name="velocity">
+                <param name="min">-10</param>
                 <param name="max">10</param>
-            </comand_interface>
+            </command_interface>
+            <state_interface name="velocity"/>
+            <state_interface name="position"/>
+        </joint>
+        <joint name="right_front_wheel_joint">
+            <command_interface name="velocity">
+                <param name="min">-10</param>
+                <param name="max">10</param>
+            </command_interface>
+            <state_interface name="velocity"/>
+            <state_interface name="position"/>
+        </joint>
+         <joint name="right_back_wheel_joint">
+            <command_interface name="velocity">
+                <param name="min">-10</param>
+                <param name="max">10</param>
+            </command_interface>
             <state_interface name="velocity"/>
             <state_interface name="position"/>
@@ -23,6 +39,6 @@
     </ros2_control>
     <gazebo>
-        <plugin name='gazebo_ros2_control' filename='libgazebo_ros2_control'>
-            <parameters>$(find centinela)/config/my_controller.yaml</parameters>
+        <plugin name='gazebo_ros2_control' filename='libgazebo_ros2_control.so'>
+            <parameters>$(find centinel)/config/my_controllers.yaml</parameters>
         </plugin>
     </gazebo>

Commit message: Main

File: description/gazebo_control.xacro (robot description, xacro)
@@ -8,5 +8,5 @@
             <left_back_joint>left_back_wheel_joint</left_joint>
             <right_back_joint>right_back_wheel_joint</right_joint>
-            <wheel_separation>0.36</wheel_separation>
+            <wheel_separation>0.40</wheel_separation>
             <wheel_diameter>0.136</wheel_diameter>
             <!-- Limits -->

File: description/robot.urdf.xacro (robot description, xacro)
@@ -1,11 +1,11 @@
 <?xml version="1.0"?>
 <robot xmlns:xacro="http://www.ros.org/wiki/xacro"  name="robot">
-    <xacro:args name="use_ros2_control" default="true"/>
+    <xacro:arg name="use_ros2_control" default="true"/>
     <xacro:include filename="robot_core.xacro"/>
-    <xacro:if value="${arg use_ros2_control}">
-    <xacro:include filename="ros2_control.xacro"/>
+    <xacro:if value="$(arg use_ros2_control)">
+        <xacro:include filename="ros2_control.xacro"/>
     </xacro:if>
-    <xacro:unless value="${arg use_ros2_control}">
-    <xacro:include filename="gazebo_control.xacro"/>
+    <xacro:unless value="$(arg use_ros2_control)">
+        <xacro:include filename="gazebo_control.xacro"/>
     </xacro:unless>
     <xacro:include filename="lidar.xacro"/>

File: description/robot_core.xacro (robot description, xacro)
@@ -51,5 +51,5 @@
         <parent link="base_link"/>
         <child link="left_front_wheel"/>
-        <origin xyz="0.1323 0.18 0.0235" rpy="-${pi/2} 0 0"/>
+        <origin xyz="0.1323 0.2 0.0235" rpy="-${pi/2} 0 0"/>
         <axis xyz="0 0 1"/>
     </joint>
@@ -76,5 +76,5 @@
         <parent link="base_link"/>
         <child link="left_back_wheel"/>
-        <origin xyz="-0.1323 0.18 0.0235" rpy="-${pi/2} 0 0"/>
+        <origin xyz="-0.1323 0.2 0.0235" rpy="-${pi/2} 0 0"/>
         <axis xyz="0 0 1"/>
     </joint>
@@ -102,5 +102,5 @@
         <parent link="base_link"/>
         <child link="right_front_wheel"/>
-        <origin xyz="0.1323 -0.18 0.0235" rpy="${pi/2} 0 0"/>
+        <origin xyz="0.1323 -0.2 0.0235" rpy="${pi/2} 0 0"/>
         <axis xyz="0 0 -1"/>
     </joint>
@@ -127,5 +127,5 @@
         <parent link="base_link"/>
         <child link="right_back_wheel"/>
-        <origin xyz="-0.1323 -0.18 0.0235" rpy="${pi/2} 0 0"/>
+        <origin xyz="-0.1323 -0.2 0.0235" rpy="${pi/2} 0 0"/>
         <axis xyz="0 0 -1"/>
     </joint>
