Commit message: add wheels

File: description/robot_core.xacro (robot description, xacro)
@@ -20,11 +20,11 @@
         <parent link="base_link"/>
         <child link="chassis" />
-        <origin xyz="-0.1 0 0"/>
+        <origin xyz="-0.2 0 0"/>
     </joint>
     <link name="chassis">
         <visual>
-            <origin xyz="-0.195 0 0.053"/>
+            <origin xyz="0.2 0 0.053"/>
             <geometry>
-                <box size="0.29 0.39 .106"/>
+                <box size="0.4 0.3 0.106"/>
             </geometry>
             <material name="white"/>
@@ -32,3 +32,32 @@
     </link>
      <!--LEFT WHELS-->
+     <joint name= "left_wheel_joint" type="continuous">
+        <parent link="base_link"/>
+        <child link="left_wheel"/>
+        <origin xyz="0.068 0.15 0" rpy="-${pi/2} 0 0"/>
+        <axis xyz="0 0 1"/>
+     </joint>
+    <link name="left_wheel">
+        <visual>
+            <geometry>
+                <cylinder radius="0.068" length="0.067"/>
+            </geometry>
+            <material name="blue"/>
+        </visual>
+    </link>
+     <!--RIGHT WHELS-->
+     <joint name= "right_wheel_joint" type="continuous">
+        <parent link="base_link"/>
+        <child link="right_wheel"/>
+        <origin xyz="0.068 -0.15 0" rpy="${pi/2} 0 0"/>
+        <axis xyz="0 0 -1"/>
+     </joint>
+    <link name="right_wheel">
+        <visual>
+            <geometry>
+                <cylinder radius="0.068" length="0.067"/>
+            </geometry>
+            <material name="blue"/>
+        </visual>
+    </link>
 </robot>

Commit message: 4 wheels axis

File: description/robot_core.xacro (robot description, xacro)
@@ -32,11 +32,25 @@
     </link>
      <!--LEFT WHELS-->
-     <joint name= "left_wheel_joint" type="continuous">
+     <joint name="left_wheel_joint" type="continuous">
         <parent link="base_link"/>
         <child link="left_wheel"/>
-        <origin xyz="0.068 0.15 0" rpy="-${pi/2} 0 0"/>
+        <origin xyz="0.1323 0.15 0" rpy="-${pi/2} 0 0"/>
         <axis xyz="0 0 1"/>
      </joint>
     <link name="left_wheel">
+        <visual>
+            <geometry>
+                <cylinder radius="0.068" length="0.067"/>
+            </geometry>
+            <material name="blue"/>
+        </visual>
+    </link>
+      <joint name="left_wheel_joint1" type="continuous">
+        <parent link="base_link"/>
+        <child link="left_wheel1"/>
+        <origin xyz="-0.1323 0.18 0" rpy="-${pi/2} 0 0"/>
+        <axis xyz="0 0 1"/>
+     </joint>
+    <link name="left_wheel1">
         <visual>
             <geometry>
@@ -50,5 +64,5 @@
         <parent link="base_link"/>
         <child link="right_wheel"/>
-        <origin xyz="0.068 -0.15 0" rpy="${pi/2} 0 0"/>
+        <origin xyz="0.1323 -0.15 0" rpy="${pi/2} 0 0"/>
         <axis xyz="0 0 -1"/>
      </joint>
@@ -61,3 +75,17 @@
         </visual>
     </link>
+     <joint name= "right_wheel_joint1" type="continuous">
+        <parent link="base_link"/>
+        <child link="right_wheel1"/>
+        <origin xyz="-0.1323 -0.15 0" rpy="${pi/2} 0 0"/>
+        <axis xyz="0 0 -1"/>
+     </joint>
+    <link name="right_wheel1">
+        <visual>
+            <geometry>
+                <cylinder radius="0.068" length="0.067"/>
+            </geometry>
+            <material name="blue"/>
+        </visual>
+    </link>
 </robot>

Commit message: slam test and config

File: description/robot_core.xacro (robot description, xacro)
@@ -19,4 +19,12 @@
         <!--BASE LINK-->
     <link name="base_link">
+    </link>
+    <!--base footprint-->
+    <joint name="base_footprint_joint" type="fixed">
+        <parent link="base_link"/>
+        <child link="base_footprint"/>
+        <origin xyz="0 0 0" rpy="0 0 0"/>
+    </joint>
+    <link name="base_footprint">
     </link>
         <!--CHASSIS LINK-->
